File: hardware/altimeter.kicad_pcb (KiCad board)
At the start: 4 copper layers, 12 x 34 mm, 39 parts, among them J1 USB_C_Receptacle_USB2.0_16P, J2 Conn_01x05_MountingPin, SW2 SW_SPDT, U1 nRF52833_QDxx, U2 MCP73832T-2, U3 BMP390L, U4 W25X40CLUXIG, U5 LIS2DH, Y1 32MHz

Commit message: new hardware revision
Parts:
- added C19: 33u, Capacitor_SMD:C_0805_2012Metric, F.Cu at (63.1, 41.8)
- moved H2 0.25 mm to (60.0, 37.8)
- moved H3 0.25 mm to (57.0, 37.8)
- moved SW2 0.25 mm to (58.5, 37.8)
- moved J2 0.20 mm to (58.5, 66.7)
- moved J1 0.16 mm to (58.5, 65.9)
Routing:
- net Earth: track 39.7 -> 43.6 mm
- net VCC: track 22.8 -> 25.7 mm
- net NRF_VDD: track 42.2 -> 43.6 mm
- net +1V8: track 24.6 -> 25.8 mm
Other:
- board text added: "V1.1"
- board text removed: "V1.0"
