File: hardware/wren_bt/altimeter2.kicad_pcb (KiCad board)
At the start: 4 copper layers, 14 x 30 mm, 13 parts, among them J1 Conn_01x03, Q1 Q_PMOS_GSD, SW2 SW_Push_Shielded, U1 E104-BT5032A, U2 BMP390L, U3 W25X40CLUXIG, U5 LSM6DS3

Commit message: orderer v1.0-bt
Parts:
- added G***: LOGO, LOGO, B.Cu at (121.1, 104.8)
Other:
- board text added: "Wren-bt 1.0 feb 2025"
Changed lines of the file:
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@@
 		(attr through_hole dnp)
 		(fp_line
-			(start -1.33 -1.33)
-			(end 0 -1.33)
-			(stroke
-				(width 0.12)
-				(type solid)
-			)
-			(layer "F.SilkS")
-		)
-		(fp_line
-			(start -1.33 0)
-			(end -1.33 -1.33)
-			(stroke
-				(width 0.12)
-				(type solid)
-			)
-			(layer "F.SilkS")
-		)
-		(fp_line
-			(start -1.33 1.27)
-			(end -1.33 6.41)
-			(stroke
-				(width 0.12)
-				(type solid)
-			)
-			(layer "F.SilkS")
-		)
-		(fp_line
-			(start -1.33 1.27)
-			(end 1.33 1.27)
-			(stroke
-				(width 0.12)
-				(type solid)
-			)
-			(layer "F.SilkS")
-		)
-		(fp_line
-			(start -1.33 6.41)
-			(end 1.33 6.41)
-			(stroke
-				(width 0.12)
-				(type solid)
-			)
-			(layer "F.SilkS")
-		)
-		(fp_line
-			(start 1.33 1.27)
-			(end 1.33 6.41)
-			(stroke
-				(width 0.12)
-				(type solid)
-			)
-			(layer "F.SilkS")
-		)
-		(fp_line
 			(start -1.8 -1.8)
 			(end -1.8 6.85)
@@
 			(unlocked yes)
 			(layer "F.SilkS")
+			(hide yes)
 			(effects
 				(font
@@
 			(at 0 -6 90)
 			(layer "B.SilkS")
+			(hide yes)
 			(effects
 				(font
@@
 		)
 	)
+	(footprint "LOGO"
+		(layer "B.Cu")
+		(at 121.127436 104.845621 180)
+		(property "Reference" "G***"
+			(at 0 0 0)
+			(layer "B.SilkS")
+			(hide yes)
+			(effects
+				(font
+					(size 1.5 1.5)
+					(thickness 0.3)
+				)
+				(justify mirror)
+			)
+		)
+		(property "Value" "LOGO"
+			(at 0.75 0 0)
+			(layer "B.SilkS")
+			(hide yes)
+			(effects
+				(font
+					(size 1.5 1.5)
+					(thickness 0.3)
+				)
+				(justify mirror)
+			)
+		)
+		(property "Footprint" ""
+			(at 0 0 0)
+			(layer "B.Fab")
+			(hide yes)
+			(effects
+				(font
+					(size 1.27 1.27)
+					(thickness 0.15)
+				)
+				(justify mirror)
+			)
+		)
+		(property "Datasheet" ""
+			(at 0 0 0)
+			(layer "B.Fab")
+			(hide yes)
+			(effects
+				(font
+					(size 1.27 1.27)
+					(thickness 0.15)
+				)
+				(justify mirror)
+			)
+		)
+		(property "Description" ""
+			(at 0 0 0)
+			(layer "B.Fab")
+			(hide yes)
+			(effects
+				(font
+					(size 1.27 1.27)
+					(thickness 0.15)
+				)
+				(justify mirror)
+			)
+		)
+		(attr board_only exclude_from_pos_files exclude_from_bom)
+		(fp_poly
+			(pts
+				(xy 0.124886 0.008933) (xy 0.151693 -0.087022) (xy 0.139919 -0.200882) (xy 0.090178 -0.290572) (xy -0.006311 -0.338409)
+				(xy -0.130848 -0.347801) (xy -0.238817 -0.32035) (xy -0.281837 -0.277203) (xy -0.265276 -0.198626)
+				(xy -0.188971 -0.100821) (xy -0.081877 -0.011165) (xy 0.027052 0.042962) (xy 0.062624 0.048515)
+			)
+			(stroke
+				(width 0)
+				(type solid)
+			)
+			(fill solid)
+			(layer "B.SilkS")
+		)
+		(fp_poly
+			(pts
+				(xy -1.016009 -0.543122) (xy -1.001972 -0.605038) (xy -0.955166 -0.744651) (xy -0.827337 -0.877079)
+				(xy -0.637367 -0.987488) (xy -0.427885 -1.055993) (xy -0.243761 -1.09004) (xy -0.093481 -1.09357)
+				(xy 0.074425 -1.065163) (xy 0.178347 -1.039255) (xy 0.458936 -0.960174) (xy 0.653584 -0.890304)
+				(xy 0.775238 -0.822715) (xy 0.836846 -0.750476) (xy 0.851677 -0.678888) (xy 0.8781 -0.575224) (xy 0.929705 -0.551085)
+				(xy 0.979011 -0.574071) (xy 0.996091 -0.657659) (xy 0.992329 -0.764004) (xy 0.976924 -0.976924)
+				(xy 0.576135 -1.11321) (xy 0.128251 -1.224195) (xy -0.297011 -1.242319) (xy -0.674617 -1.178937)
+				(xy -0.914203 -1.078038) (xy -1.074198 -0.928804) (xy -1.147953 -0.738273) (xy -1.152268 -0.673538)
+				(xy -1.135422 -0.54496) (xy -1.081947 -0.501142) (xy -1.07712 -0.500987)
+			)
+			(stroke
+				(width 0)
+				(type solid)
+			)
+			(fill solid)
+			(layer "B.SilkS")
+		)
+		(fp_poly
+			(pts
+				(xy -0.489389 1.884673) (xy -0.214455 1.862298) (xy 0.068712 1.82165) (xy 0.330847 1.766171) (xy 0.542684 1.699299)
+				(xy 0.568081 1.6886) (xy 0.817057 1.535688) (xy 1.068028 1.302958) (xy 1.304521 1.009073) (xy 1.510066 0.672697)
+				(xy 1.568567 0.554974) (xy 1.661369 0.352492) (xy 1.718025 0.204238) (xy 1.745724 0.074096) (xy 1.751657 -0.074048)
+				(xy 1.743012 -0.276309) (xy 1.741028 -0.311351) (xy 1.723979 -0.540033) (xy 1.697804 -0.702842)
+				(xy 1.653258 -0.834103) (xy 1.581094 -0.96814) (xy 1.551039 -1.016621) (xy 1.435887 -1.20278) (xy 1.320654 -1.394837)
+				(xy 1.264315 -1.49174) (xy 1.18494 -1.618738) (xy 1.100935 -1.714692) (xy 0.997227 -1.784181) (xy 0.858747 -1.831789)
+				(xy 0.670421 -1.862096) (xy 0.41718 -1.879683) (xy 0.083952 -1.889133) (xy -0.050098 -1.891304)
+				(xy -0.404284 -1.894096) (xy -0.671702 -1.890332) (xy -0.865609 -1.879289) (xy -0.999264 -1.860244)
+				(xy -1.080312 -1.835076) (xy -1.253177 -1.717757) (xy -1.430525 -1.530402) (xy -1.590741 -1.299716)
+				(xy -1.710807 -1.056047) (xy -1.792812 -0.755161) (xy -1.83788 -0.392311) (xy -1.845362 -0.061373)
+				(xy -1.753451 -0.061373) (xy -1.753451 -0.275903) (xy -1.725727 -0.523797) (xy -1.650941 -0.812891)
+				(xy -1.541677 -1.103873) (xy -1.410517 -1.357432) (xy -1.40393 -1.367919) (xy -1.297888 -1.51685)
+				(xy -1.184208 -1.627842) (xy -1.046604 -1.706186) (xy -0.868793 -1.757172) (xy -0.634491 -1.786091)
+				(xy -0.327412 -1.798234) (xy -0.075147 -1.799623) (xy 0.241871 -1.794645) (xy 0.513151 -1.782045)
+				(xy 0.720719 -1.763021) (xy 0.846598 -1.738769) (xy 0.84856 -1.7381) (xy 0.979897 -1.665301) (xy 1.102268 -1.531814)
+				(xy 1.187055 -1.402762) (xy 1.300195 -1.215639) (xy 1.414719 -1.026812) (xy 1.478141 -0.922591)
+				(xy 1.55698 -0.748018) (xy 1.614121 -0.53531) (xy 1.644517 -0.318159) (xy 1.64312 -0.130258) (xy 1.613475 -0.019281)
+				(xy 1.547154 0.040354) (xy 1.406482 0.126594) (xy 1.210157 0.228878) (xy 1.006033 0.323846) (xy 0.76258 0.437338)
+				(xy 0.581857 0.533851) (xy 0.47529 0.606844) (xy 0.450888 0.641579) (xy 0.484987 0.688244) (xy 0.590027 0.684531)
+				(xy 0.770124 0.629441) (xy 1.029393 0.521974) (xy 1.128931 0.476738) (xy 1.305747 0.397302) (xy 1.443865 0.339472)
+				(xy 1.521561 0.312172) (xy 1.530771 0.311703) (xy 1.518857 0.360553) (xy 1.47341 0.472045) (xy 1.424179 0.579667)
+				(xy 1.308469 0.777145) (xy 1.146447 0.994717) (xy 0.960294 1.207631) (xy 0.77219 1.391133) (xy 0.604316 1.520468)
+				(xy 0.557513 1.546858) (xy 0.400551 1.605392) (xy 0.180245 1.663405) (xy -0.07437 1.715888) (xy -0.334258 1.757832)
+				(xy -0.570382 1.784226) (xy -0.753706 1.790063) (xy -0.815921 1.783814) (xy -0.955999 1.721679)
+				(xy -1.12291 1.594688) (xy -1.293763 1.424975) (xy -1.445667 1.234673) (xy -1.535095 1.088464) (xy -1.580071 0.972025)
+				(xy -1.633243 0.793362) (xy -1.685493 0.588943) (xy -1.727702 0.395233) (xy -1.750753 0.2487) (xy -1.752581 0.218676)
+				(xy -1.708894 0.205268) (xy -1.583867 0.229538) (xy -1.388068 0.289257) (xy -1.340138 0.305679)
+				(xy -1.066707 0.394111) (xy -0.875165 0.439288) (xy -0.757459 0.442117) (xy -0.705537 0.403504)
+				(xy -0.70138 0.37767) (xy -0.747891 0.317103) (xy -0.873552 0.262004) (xy -0.914299 0.250688) (xy -1.0773 0.201692)
+				(xy -1.281543 0.129809) (xy -1.440335 0.067775) (xy -1.753451 -0.061373) (xy -1.845362 -0.061373)
+				(xy -1.846786 0.001636) (xy -1.820301 0.395813) (xy -1.759198 0.759353) (xy -1.664251 1.06139) (xy -1.657389 1.07712)
+				(xy -1.539481 1.282815) (xy -1.377028 1.489307) (xy -1.19371 1.672177) (xy -1.013204 1.807001) (xy -0.897491 1.860851)
+				(xy -0.726823 1.885338)
+			)
+			(stroke
+				(width 0)
+				(type solid)
+			)
+			(fill solid)
+			(layer "B.SilkS")
+		)
+	)
 	(gr_circle
 		(center 114.5 107)
@@
 		(layer "Edge.Cuts")
 	)
+	(gr_text "Wren-bt 1.0\nfeb 2025\n"
+		(at 118.625 83.475 0)
+		(layer "B.SilkS")
+		(effects
+			(font
+				(size 1 1)
+				(thickness 0.15)
+			)
+			(justify bottom mirror)
+		)
+	)
 	(segment
